Commit message: Transfer checkpoint: gripper fixes + middleware updates + trajectory system improvements

File: src/dexter_arm_description/urdf/dexter_arm.urdf.xacro (robot description, xacro)
@@ -270,5 +270,5 @@
         <child link="l6l_finger_slider" />
         <axis xyz="0 0 1" />
-        <limit lower="-0.04" upper="0.0" effort="1.0" velocity="0.1" />
+        <limit lower="-0.02" upper="0.0" effort="1.0" velocity="0.1" />
     </joint>
     <!-- LEFT GRIPPER - Finger (actual mesh) -->
@@ -306,5 +306,5 @@
         <child link="l6l_finger2_slider" />
         <axis xyz="0 0 1" />
-        <limit lower="-0.04" upper="0.0" effort="1.0" velocity="0.1" />
+        <limit lower="-0.02" upper="0.0" effort="1.0" velocity="0.1" />
     </joint>
     <!-- LEFT GRIPPER - Second Finger (actual mesh) -->
@@ -607,5 +607,5 @@
         <child link="l6r_finger_slider" />
         <axis xyz="0 0 1" />
-        <limit lower="-0.022" upper="0.0" effort="10.0" velocity="0.1" />
+        <limit lower="-0.020" upper="0.0" effort="10.0" velocity="0.1" />
     </joint>
     <!-- RIGHT GRIPPER - Finger (actual mesh) -->
@@ -649,5 +649,5 @@
         <child link="l6r_finger2_slider" />
         <axis xyz="0 0 1" />
-        <limit lower="-0.022" upper="0.022" effort="10.0" velocity="0.1" />
+        <limit lower="0" upper="0.020" effort="10.0" velocity="0.1" />
     </joint>
     <!-- RIGHT GRIPPER - Second Finger (actual mesh) -->
