Commit message: feat(trajectory): add execution context differentiation (hardware/gazebo/simulated)
- Add execution_context field to RobotState to track execution backend
- Update _run_trajectory to accept context parameter and enhance logging
- Update execute_trajectory to auto-detect execution context based on running sessions
- Add execution context to snapshot payload
- Update Shape tab to display and track execution context
- All Shape Generation (main) tab features now complete with full lifecycle

File: src/dexter_arm_description/urdf/dexter.urdf (robot description, URDF)
Before this commit: robot dexter_arm, 28 links, 27 joints
Joints:
- joint j1l: limit lower=0 upper=3.14 effort=343.0 velocity=5 -> lower=-1.57 upper=1.57 effort=343.0 velocity=5
- joint j1r: limit lower=0 upper=3.14 effort=343.0 velocity=5 -> lower=-1.57 upper=1.57 effort=343.0 velocity=5

File: src/dexter_arm_description/urdf/dexter_arm.urdf.xacro (robot description, xacro)
@@ -64,5 +64,5 @@
         <child link="l1l" />
         <axis xyz="0 0 -1" />
-        <limit lower="0" upper="3.14" effort="343.0" velocity="5" />
+        <limit lower="-1.57" upper="1.57" effort="343.0" velocity="5" />
     </joint>
     <!-- Link l2l -->
@@ -206,10 +206,4 @@
             </material>
         </visual>
-        <collision>
-            <origin xyz="0 0 0" rpy="0 0 0" />
-            <geometry>
-                <mesh filename="package://dexter_arm_description/meshes/base.stl" scale="0.001 0.001 0.001"/>
-            </geometry>
-        </collision>
     </link>
     <joint name="j6l" type="revolute">
@@ -236,10 +230,4 @@
             </material>
         </visual>
-        <collision>
-            <origin xyz="0 0 0" rpy="0 0 0" />
-            <geometry>
-                <mesh filename="package://dexter_arm_description/meshes/base1.stl" scale="0.001 0.001 0.001"/>
-            </geometry>
-        </collision>
     </link>
     <joint name="j6l_base1_fixed" type="fixed">
@@ -264,10 +252,4 @@
             </material>
         </visual>
-        <collision>
-            <origin xyz="0 0 0" rpy="0 0 0" />
-            <geometry>
-                <mesh filename="package://dexter_arm_description/meshes/rail.stl" scale="0.001 0.001 0.001"/>
-            </geometry>
-        </collision>
     </link>
     <joint name="j6l_rail_fixed" type="fixed">
@@ -288,5 +270,5 @@
         <child link="l6l_finger_slider" />
         <axis xyz="0 0 1" />
-        <limit lower="-0.022" upper="0.0" effort="1.0" velocity="0.1" />
+        <limit lower="-0.04" upper="0.0" effort="1.0" velocity="0.1" />
     </joint>
     <!-- LEFT GRIPPER - Finger (actual mesh) -->
@@ -306,10 +288,4 @@
             </material>
         </visual>
-        <collision>
-            <origin xyz="0 0 0" rpy="0 0 0" />
-            <geometry>
-                <mesh filename="package://dexter_arm_description/meshes/finger.stl" scale="0.001 0.001 0.001"/>
-            </geometry>
-        </collision>
     </link>
     <joint name="j6l_finger_fixed" type="fixed">
@@ -330,5 +306,5 @@
         <child link="l6l_finger2_slider" />
         <axis xyz="0 0 1" />
-        <limit lower="-0.022" upper="0.0" effort="1.0" velocity="0.1" />
+        <limit lower="-0.04" upper="0.0" effort="1.0" velocity="0.1" />
     </joint>
     <!-- LEFT GRIPPER - Second Finger (actual mesh) -->
@@ -348,10 +324,4 @@
             </material>
         </visual>
-        <collision>
-            <origin xyz="0 0 0" rpy="0 0 0" />
-            <geometry>
-                <mesh filename="package://dexter_arm_description/meshes/finger.stl" scale="0.001 0.001 0.001"/>
-            </geometry>
-        </collision>
     </link>
     <joint name="j6l_finger2_fixed" type="fixed">
@@ -376,10 +346,4 @@
             </material>
         </visual>
-        <collision>
-            <origin xyz="0 0 0" rpy="0 0 0" />
-            <geometry>
-                <sphere radius="0.008" />
-            </geometry>
-        </collision>
     </link>
     <joint name="tool0_left_fixed_joint" type="fixed">
@@ -418,5 +382,5 @@
         <child link="l1r" />
         <axis xyz="0 0 1" />
-        <limit lower="0" upper="3.14" effort="343.0" velocity="5" />
+        <limit lower="-1.57" upper="1.57" effort="343.0" velocity="5" />
     </joint>
     <!-- Link l2r -->
@@ -731,10 +695,4 @@
             </material>
         </visual>
-        <collision>
-            <origin xyz="0 0 0" rpy="0 0 0" />
-            <geometry>
-                <sphere radius="0.008" />
-            </geometry>
-        </collision>
     </link>
     <joint name="tool0_right_fixed_joint" type="fixed">

File: src/dexter_arm_hardware/urdf/dexter_arm_hardware.xacro (robot description, xacro)
@@ -62,5 +62,5 @@
       <joint name="j7l1">
         <command_interface name="position">
-          <param name="min">-0.022</param>
+          <param name="min">-0.04</param>
           <param name="max">0.0</param>
         </command_interface>
@@ -70,5 +70,5 @@
       <joint name="j7l2">
         <command_interface name="position">
-          <param name="min">-0.022</param>
+          <param name="min">-0.04</param>
           <param name="max">0.0</param>
         </command_interface>

Commit message: Fix: Right arm joint inversion sync issue in ESP32 firmware
- Added missing inversion logic for right arm joints (8, 9, 10, 11) in command_callback
- Right arm joints are mechanically mirrored with reversed Z-axis vs left arm
- Gripper controller was syncing fine (no inversion needed) but arm controller was out of sync
- Now both left arm (indices 1, 3, 4) and right arm (indices 8, 9, 10, 11) properly invert commands
- This fixes the hardware sync mismatch where arm commands were going in opposite direction

Changes:
- esp32_firmware_wireless.ino: Updated joint inversion logic for symmetry
- Also includes gripper execution fixes, URDF/SRDF updates, and UI enhancements from previous work

File: src/dexter_arm_description/urdf/dexter.urdf (robot description, URDF)
Before this commit: robot dexter_arm, 28 links, 27 joints
Links:
- removed link l6l_base1
- removed link l6l_finger
- removed link l6l_finger2
- removed link l6l_finger2_slider
- removed link l6l_finger_slider
- removed link l6l_rail
- removed link l6r_base1
- removed link l6r_finger
- removed link l6r_finger2
- removed link l6r_finger2_slider
- removed link l6r_finger_slider
- removed link l6r_rail
- removed link tool0_left
- removed link tool0_right
- removed link world
- added link l7l1, mass 0.0508689051828396; collision mesh filename=package://dexter_arm_description/meshes/l7l1.STL; visual mesh filename=package://dexter_arm_description/meshes/l7l1.STL
- added link l7l2, mass 0.0508689051828397; collision mesh filename=package://dexter_arm_description/meshes/l7l2.STL; visual mesh filename=package://dexter_arm_description/meshes/l7l2.STL
- added link l7r1, mass 0.0508689051689457; collision mesh filename=package://dexter_arm_description/meshes/l7r1.STL; visual mesh filename=package://dexter_arm_description/meshes/l7r1.STL
- added link l7r2, mass 0.0508689051828396; collision mesh filename=package://dexter_arm_description/meshes/l7r2.STL; visual mesh filename=package://dexter_arm_description/meshes/l7r2.STL
- link base_link: mass 1.57034512332414 -> 1.50541140238431; geometry collision mesh filename=package://dexter_arm_description/meshes/base_link.STL; visual mesh filename=package://dexter_arm_description/meshes/base_link.STL
- link l1l: geometry collision mesh filename=package://dexter_arm_description/meshes/l1l.STL; visual mesh filename=package://dexter_arm_description/meshes/l1l.STL
- link l1r: mass 0.0412610106656879 -> 0.0412610106656878; geometry collision mesh filename=package://dexter_arm_description/meshes/l1r.STL; visual mesh filename=package://dexter_arm_description/meshes/l1r.STL
- link l2l: mass 0.0412639771770677 -> 0.0412639771770678; geometry collision mesh filename=package://dexter_arm_description/meshes/l2l.STL; visual mesh filename=package://dexter_arm_description/meshes/l2l.STL
- link l2r: geometry collision mesh filename=package://dexter_arm_description/meshes/l2r.STL; visual mesh filename=package://dexter_arm_description/meshes/l2r.STL
- link l3l: mass 0.089584582698146 -> 0.0895845826981461; geometry collision mesh filename=package://dexter_arm_description/meshes/l3l.STL; visual mesh filename=package://dexter_arm_description/meshes/l3l.STL
- link l3r: geometry collision mesh filename=package://dexter_arm_description/meshes/l3r.STL; visual mesh filename=package://dexter_arm_description/meshes/l3r.STL
- link l4l: mass 0.041263977177068 -> 0.0412639771770679; geometry collision mesh filename=package://dexter_arm_description/meshes/l4l.STL; visual mesh filename=package://dexter_arm_description/meshes/l4l.STL
- link l4r: mass 0.0412639771770679 -> 0.0412639771770678; geometry collision mesh filename=package://dexter_arm_description/meshes/l4r.STL; visual mesh filename=package://dexter_arm_description/meshes/l4r.STL
- link l5l: mass 0.0877350527785506 -> 0.0877350527785504; geometry collision mesh filename=package://dexter_arm_description/meshes/l5l.STL; visual mesh filename=package://dexter_arm_description/meshes/l5l.STL
- link l5r: mass 0.0877350517033452 -> 0.0877350527785506; geometry collision mesh filename=package://dexter_arm_description/meshes/l5r.STL; visual mesh filename=package://dexter_arm_description/meshes/l5r.STL
- link l6l: mass 0.05 -> 0.160590985030217; geometry collision mesh filename=package://dexter_arm_description/meshes/l6l.STL; visual mesh filename=package://dexter_arm_description/meshes/l6l.STL
- link l6r: mass 0.05 -> 0.160590985030217; geometry collision mesh filename=package://dexter_arm_description/meshes/l6r.STL; visual mesh filename=package://dexter_arm_description/meshes/l6r.STL
Joints:
- removed joint base_joint
- removed joint j6l_base1_fixed
- removed joint j6l_finger2_fixed
- removed joint j6l_finger_fixed
- removed joint j6l_rail_fixed
- removed joint j6r_base1_fixed
- removed joint j6r_finger2_fixed
- removed joint j6r_finger_fixed
- removed joint j6r_rail_fixed
- removed joint tool0_left_fixed_joint
- removed joint tool0_right_fixed_joint
- joint j1l: axis 0 0 -1 -> 0 0 1; limit lower=-1.57 upper=1.57 effort=343.0 velocity=5 -> lower=-1.57 upper=1.57 effort=3.43 velocity=5; origin xyz=-0.185 0 0.4755 rpy=0 0 0 -> xyz=-0.185 0 0.5347 rpy=3.14159265358979 0 0
- joint j1r: limit lower=-1.57 upper=1.57 effort=343.0 velocity=5 -> lower=-1.57 upper=1.57 effort=3.43 velocity=5; origin xyz=0.185 0 0.4755 rpy=3.14159265358979 0 0 -> xyz=0.185 0 0.534699999999999 rpy=-3.14159265358979 0 0
- joint j2l: limit lower=-1.57 upper=1.57 effort=343.0 velocity=5 -> lower=-1.57 upper=1.57 effort=3.43 velocity=5; origin xyz=0 0 0.01 rpy=0 1.5707963267949 0 -> xyz=0 0 0.0340000000000011 rpy=0 -1.5707963267949 0
- joint j2r: axis 0 0 1 -> 0 0 -1; limit lower=-1.57 upper=1.57 effort=343.0 velocity=5 -> lower=-1.57 upper=1.57 effort=3.43 velocity=5; origin xyz=0 0 -0.01 rpy=0 -1.5707963267949 0 -> xyz=0 0 0.0339999999999996 rpy=3.14159265358979 -1.5707963267949 0
- joint j3l: limit lower=-1.57 upper=1.57 effort=343.0 velocity=5 -> lower=-1.57 upper=1.57 effort=3.43 velocity=5; origin xyz=0.0839999999999997 0 0 rpy=0 0 0 -> xyz=0.083999999999998 0 0 rpy=0 0 0
- joint j3r: axis 0.000972696716171088 1.23048895120007E-05 0.999999526854732 -> 0 0 -1; limit lower=-1.57 upper=1.57 effort=343.0 velocity=5 -> lower=-1.57 upper=1.57 effort=3.43 velocity=5; origin xyz=0.0839999999999999 0 0 rpy=1.23048953327578E-05 -0.00097269686955413 -0.012649615042804 -> xyz=0.0840000000000007 0 0 rpy=0 0 0
- joint j4l: limit lower=-1.57 upper=1.57 effort=147.0 velocity=5 -> lower=-1.57 upper=1.57 effort=1.5 velocity=5; origin xyz=0.0849999999944108 0 0 rpy=0 0 0 -> xyz=0.0850000000000001 0 0 rpy=0 0 0
- joint j4r: axis 0.000972696716170201 1.23048895400181E-05 0.999999526854732 -> 0 0 -1; limit lower=-1.57 upper=1.57 effort=147.0 velocity=5 -> lower=-1.57 upper=1.57 effort=1.5 velocity=5; origin xyz=0.0849931593404333 0.00107518760394861 -8.26858361745036E-05 rpy=0 0 0 -> xyz=0.0850000000000011 0 0 rpy=0 0 0
- joint j5l: limit lower=-1.57 upper=1.57 effort=147.0 velocity=5 -> lower=-1.57 upper=1.57 effort=1.5 velocity=5; origin xyz=0.083965824229058 0.0023959051595066 0 rpy=0 0 0 -> xyz=0.0840000000000015 0 0 rpy=0 0 0
- joint j5r: axis 0.000769310840231528 0 0.999999704050751 -> 0 0 -1; limit lower=-1.57 upper=1.57 effort=147.0 velocity=5 -> lower=-1.57 upper=1.57 effort=1.5 velocity=5; origin xyz=0.0839932398190739 0.00106253831537445 -8.1713061631225E-05 rpy=0 0.000203415098013994 0.00264506784365567 -> xyz=0.083999999999999 0 0 rpy=0 0 0
- joint j6l: axis 0 0 1 -> 0 0 -1; limit lower=-1.5708 upper=1.5708 effort=0.5 velocity=1.0 -> lower=-3.14 upper=3.14 effort=1.5 velocity=5; origin xyz=0.110 -0.002 0.010 rpy=3.14159 1.57 0 -> xyz=0.100000000000004 0.00011000000184596 -0.0115000000043161 rpy=0 1.5707963267949 0
- joint j6r: axis 0 0 1 -> 0 0 -1; limit lower=-1.5708 upper=1.5708 effort=0.5 velocity=1.0 -> lower=-3.14 upper=3.14 effort=1.5 velocity=5; origin xyz=0.110 0.002 0.010 rpy=3.14159 1.57 0 -> xyz=0.0999999999999998 -0.000110000000436546 0.0115000000043133 rpy=0 1.5707963267949 0
- joint j7l1: axis 0 0 1 -> 1 0 0; child l6l_finger_slider -> l7l1; limit lower=-0.022 upper=0.0 effort=1.0 velocity=0.1 -> lower=0.00 upper=-0.025 effort=0 velocity=0; origin xyz=0.000 0.022 0.021 rpy=0 -1.572 0 -> xyz=-0.00031015564213932 -0.0334996810602779 0.024487500081954 rpy=-1.5707963267949 0 0; parent l6l_rail -> l6l
- joint j7l2: axis 0 0 1 -> -1 0 0; child l6l_finger2_slider -> l7l2; limit lower=-0.022 upper=0.0 effort=1.0 velocity=0.1 -> lower=-0.025 upper=0.0 effort=0 velocity=0; origin xyz=0.060 0.022 0.021 rpy=0 1.572 0 -> xyz=0.0138251055330376 0.0320003186418183 0.0244125000819536 rpy=-1.5707963267949 0 3.14159265358979; parent l6l_rail -> l6l
- joint j7r1: axis 0 0 1 -> -1 0 0; child l6r_finger_slider -> l7r1; limit lower=-0.022 upper=0.0 effort=10.0 velocity=0.1 -> lower=-0.025 upper=0.0 effort=0 velocity=0; origin xyz=0.000 0.022 0.021 rpy=0 -1.572 0 -> xyz=0.0138251055330352 0.0320003186428659 0.0244125000819573 rpy=-1.5707963267949 0 3.14159265358979; parent l6r_rail -> l6r
- joint j7r2: axis 0 0 1 -> 1 0 0; child l6r_finger2_slider -> l7r2; limit lower=-0.022 upper=0.022 effort=10.0 velocity=0.1 -> lower=0.00 upper=-0.025 effort=0 velocity=0; origin xyz=0.060 0.022 0.021 rpy=0 -1.572 0 -> xyz=-0.000310155642144982 -0.0334996810589849 0.0244125000819576 rpy=-1.5707963267949 0 0; parent l6r_rail -> l6r
