Commit message: Fix: Right arm joint inversion sync issue in ESP32 firmware
- Added missing inversion logic for right arm joints (8, 9, 10, 11) in command_callback
- Right arm joints are mechanically mirrored with reversed Z-axis vs left arm
- Gripper controller was syncing fine (no inversion needed) but arm controller was out of sync
- Now both left arm (indices 1, 3, 4) and right arm (indices 8, 9, 10, 11) properly invert commands
- This fixes the hardware sync mismatch where arm commands were going in opposite direction

Changes:
- esp32_firmware_wireless.ino: Updated joint inversion logic for symmetry
- Also includes gripper execution fixes, URDF/SRDF updates, and UI enhancements from previous work

File: src/dexter_arm_description/urdf/dexter_arm.urdf.xacro (robot description, xacro)
@@ -1,703 +1,1042 @@
-<?xml version="1.0"?>
-<robot xmlns:xacro="http://www.ros.org/wiki/xacro" name="dexter_arm">
-    <!-- Pure robot geometry - NO ros2_control here -->
-    <!-- ros2_control is added by overlay xacros (gazebo/hardware) -->
-    <!-- Add dummy world link and fixed base_joint so base_link is not the URDF root -->
-    <link name="world" />
-    <joint name="base_joint" type="fixed">
-        <parent link="world" />
-        <child link="base_link" />
-        <origin rpy="0 0 0" xyz="0 0 0" />
-    </joint>
-    <!-- Base Link -->
-    <link name="base_link">
-        <inertial>
-            <origin xyz="1.11022302462516E-16 -1.31752248000438E-15 0.341229394008098" rpy="0 0 0" />
-            <mass value="1.57034512332414" />
-            <inertia ixx="0.014156986279529" ixy="-2.66546726272844E-17" ixz="8.0299293210262E-19"
-                     iyy="0.0167394307342646" iyz="5.42683623685501E-17" izz="0.00265284502209648" />
-        </inertial>
-        <visual>
-            <origin xyz="0 0 0" rpy="0 0 0" />
-            <geometry>
-                <mesh filename="package://dexter_arm_description/meshes/visual/base_link.STL" />
-            </geometry>
-            <material name="">
-                <color rgba="0.792156862745098 0.819607843137255 0.933333333333333 1" />
-            </material>
-        </visual>
-        <collision>
-            <origin xyz="0 0 0" rpy="0 0 0" />
-            <geometry>
-                <mesh filename="package://dexter_arm_description/meshes/collision/base_link.STL" />
-            </geometry>
-        </collision>
-    </link>
-    <!-- LEFT ARM -->
-    <!-- Link l1l -->
-    <link name="l1l">
-        <inertial>
-            <origin xyz="-2.06768076424502E-05 2.03830008427275E-15 0.0236812970530658" rpy="0 0 0" />
-            <mass value="0.0412610106656879" />
-            <inertia ixx="6.45452263055135E-06" ixy="-6.35156631471509E-20" ixz="5.67173895654462E-10"
-                     iyy="1.08529418395194E-05" iyz="1.55844839681327E-20" izz="8.35698735982534E-06" />
-        </inertial>
-        <visual>
-            <origin xyz="0 0 0" rpy="0 0 0" />
-            <geometry>
-                <mesh filename="package://dexter_arm_description/meshes/visual/l1l.STL" />
-            </geometry>
-            <material name="">
-                <color rgba="1 1 1 1" />
-            </material>
-        </visual>
-        <collision>
-            <origin xyz="0 0 0" rpy="0 0 0" />
-            <geometry>
-                <mesh filename="package://dexter_arm_description/meshes/collision/l1l.STL" />
-            </geometry>
-        </collision>
-    </link>
-    <joint name="j1l" type="revolute">
-        <origin xyz="-0.185 0 0.4755" rpy="0 0 0" />
-        <parent link="base_link" />
-        <child link="l1l" />
-        <axis xyz="0 0 -1" />
-        <limit lower="-1.57" upper="1.57" effort="343.0" velocity="5" />
-    </joint>
-    <!-- Link l2l -->
-    <link name="l2l">
-        <inertial>
-            <origin xyz="0.0420000000000009 3.10255293678452E-14 -2.1094237467878E-15" rpy="0 0 0" />
-            <mass value="0.0412639771770677" />
-            <inertia ixx="2.03861872352237E-05" ixy="1.83850917637208E-20" ixz="1.29909905427445E-20"
-                     iyy="2.30212674355657E-05" iyz="-5.99177000134609E-22" izz="8.54833447441493E-06" />
-        </inertial>
-        <visual>
-            <origin xyz="0 0 0" rpy="0 0 0" />
-            <geometry>
-                <mesh filename="package://dexter_arm_description/meshes/visual/l2l.STL" />
-            </geometry>
-            <material name="">
-                <color rgba="1 1 1 1" />
-            </material>
-        </visual>
-        <collision>
-            <origin xyz="0 0 0" rpy="0 0 0" />
-            <geometry>
-                <mesh filename="package://dexter_arm_description/meshes/collision/l2l.STL" />
-            </geometry>
-        </collision>
-    </link>
-    <joint name="j2l" type="revolute">
-        <origin xyz="0 0 0.01" rpy="0 1.5707963267949 0" />
-        <parent link="l1l" />
-        <child link="l2l" />
-        <axis xyz="0 0 1" />
-        <limit lower="-1.57" upper="1.57" effort="343.0" velocity="5" />
-    </joint>
-    <!-- Link l3l -->
-    <link name="l3l">
-        <inertial>
-            <origin xyz="0.0425000000000011 -3.91231348532972E-10 -2.05391259555654E-15" rpy="0 0 0" />
-            <mass value="0.089584582698146" />
-            <inertia ixx="1.79494942674491E-05" ixy="-6.24250401827857E-21" ixz="-1.13434779133657E-09"
-                     iyy="2.28721177257845E-05" iyz="-4.51664802349514E-21" izz="1.35465501240485E-05" />
-        </inertial>
-        <visual>
-            <origin xyz="0 0 0" rpy="0 0 0" />
-            <geometry>
-                <mesh filename="package://dexter_arm_description/meshes/visual/l3l.STL" />
-            </geometry>
-            <material name="">
-                <color rgba="1 1 1 1" />
-            </material>
-        </visual>
-        <collision>
-            <origin xyz="0 0 0" rpy="0 0 0" />
-            <geometry>
-                <mesh filename="package://dexter_arm_description/meshes/collision/l3l.STL" />
-            </geometry>
-        </collision>
-    </link>
-    <joint name="j3l" type="revolute">
-        <origin xyz="0.0839999999999997 0 0" rpy="0 0 0" />
-        <parent link="l2l" />
-        <child link="l3l" />
-        <axis xyz="0 0 1" />
-        <limit lower="-1.57" upper="1.57" effort="343.0" velocity="5" />
-    </joint>
-    <!-- Link l4l -->
-    <link name="l4l">
-        <inertial>
-            <origin xyz="0.042000000005591 -9.7518096834389E-07 -1.55431223447522E-15" rpy="0 0 0" />
-            <mass value="0.041263977177068" />
-            <inertia ixx="2.03861872352239E-05" ixy="-2.09421927761261E-21" ixz="-3.48729676766912E-20"
-                     iyy="2.3021267435566E-05" iyz="-4.08634235879589E-21" izz="8.54833447441504E-06" />
-        </inertial>
-        <visual>
-            <origin xyz="0 0 0" rpy="0 0 0" />
-            <geometry>
-                <mesh filename="package://dexter_arm_description/meshes/visual/l4l.STL" />
-            </geometry>
-            <material name="">
-                <color rgba="1 1 1 1" />
-            </material>
-        </visual>
-        <collision>
-            <origin xyz="0 0 0" rpy="0 0 0" />
-            <geometry>
-                <mesh filename="package://dexter_arm_description/meshes/collision/l4l.STL" />
-            </geometry>
-        </collision>
-    </link>
-    <joint name="j4l" type="revolute">
-        <origin xyz="0.0849999999944108 0 0" rpy="0 0 0" />
-        <parent link="l3l" />
-        <child link="l4l" />
-        <axis xyz="0 0 1" />
-        <limit lower="-1.57" upper="1.57" effort="147.0" velocity="5" />
-    </joint>
-    <!-- Link l5l -->
-    <link name="l5l">
-        <inertial>
-            <origin xyz="0.04514989228191 -0.00246541434401295 0.000519380260867508" rpy="0 0 0" />
-            <mass value="0.0877350527785506" />
-            <inertia ixx="2.15592269641528E-05" ixy="1.08634480270297E-12" ixz="6.61837513500229E-07"
-                     iyy="4.21271739710682E-05" iyz="-2.81945782664923E-12" izz="2.9808063539004E-05" />
-        </inertial>
-        <visual>
-            <origin xyz="0 0 0" rpy="0 0 0" />
-            <geometry>
-                <mesh filename="package://dexter_arm_description/meshes/visual/l5l.STL" />
-            </geometry>
-            <material name="">
-                <color rgba="1 1 1 1" />
-            </material>
-        </visual>
-        <collision>
-            <origin xyz="0 0 0" rpy="0 0 0" />
-            <geometry>
-                <mesh filename="package://dexter_arm_description/meshes/collision/l5l.STL" />
-            </geometry>
-        </collision>
-    </link>
-    <joint name="j5l" type="revolute">
-        <origin xyz="0.083965824229058 0.0023959051595066 0" rpy="0 0 0" />
-        <parent link="l4l" />
-        <child link="l5l" />
-        <axis xyz="0 0 1" />
-        <limit lower="-1.57" upper="1.57" effort="147.0" velocity="5" />
-    </joint>
-    <!-- LEFT GRIPPER BASE - Using new gripper mesh -->
-    <link name="l6l">
-        <inertial>
-            <origin xyz="0 0 0.02" rpy="0 0 0" />
-            <mass value="0.05" />
-            <inertia ixx="0.00001" ixy="0" ixz="0" iyy="0.00001" iyz="0" izz="0.00001" />
-        </inertial>
-        <visual>
-            <origin xyz="0 0 0" rpy="0 0 0" />
-            <geometry>
-                <mesh filename="package://dexter_arm_description/meshes/base.stl" scale="0.001 0.001 0.001"/>
-            </geometry>
-            <material name="">
-                <color rgba="0.5 0.5 0.5 1" />
-            </material>
-        </visual>
-    </link>
-    <joint name="j6l" type="revolute">
-        <origin xyz="0.110 -0.002 0.010" rpy="3.14159 1.57 0" />
-        <parent link="l5l" />
-        <child link="l6l" />
-        <axis xyz="0 0 1" />
-        <limit lower="-1.5708" upper="1.5708" effort="0.5" velocity="1.0" />
-    </joint>
-    <!-- LEFT GRIPPER - Base1 Layer (fixed below base) -->
-    <link name="l6l_base1">
-        <inertial>
-            <origin xyz="0 0 0.01" rpy="0 0 0" />
-            <mass value="0.03" />
-            <inertia ixx="0.00001" ixy="0" ixz="0" iyy="0.00001" iyz="0" izz="0.00001" />
-        </inertial>
-        <visual>
-            <origin xyz="0 0 0" rpy="0 0 0" />
-            <geometry>
-                <mesh filename="package://dexter_arm_description/meshes/base1.stl" scale="0.001 0.001 0.001"/>
-            </geometry>
-            <material name="">
-                <color rgba="0.5 0.5 0.5 1" />
-            </material>
-        </visual>
-    </link>
-    <joint name="j6l_base1_fixed" type="fixed">
-        <origin xyz="-0.021 0.015 0.004" rpy="3.142 0 0" />
-        <parent link="l6l" />
-        <child link="l6l_base1" />
-    </joint>
-    <!-- LEFT GRIPPER - Rail Layer (fixed to base1) -->
-    <link name="l6l_rail">
-        <inertial>
-            <origin xyz="0 0 0.01" rpy="0 0 0" />
-            <mass value="0.02" />
-            <inertia ixx="0.00001" ixy="0" ixz="0" iyy="0.00001" iyz="0" izz="0.00001" />
-        </inertial>
-        <visual>
-            <origin xyz="0 0 0" rpy="0 0 0" />
-            <geometry>
-                <mesh filename="package://dexter_arm_description/meshes/rail.stl" scale="0.001 0.001 0.001"/>
-            </geometry>
-            <material name="">
-                <color rgba="0.5 0.5 0.5 1" />
-            </material>
-        </visual>
-    </link>
-    <joint name="j6l_rail_fixed" type="fixed">
-        <origin xyz="-0.009 0.034 0.036" rpy="1.57 0 0" />
-        <parent link="l6l_base1" />
-        <child link="l6l_rail" />
-    </joint>
-    <!-- LEFT GRIPPER - Finger 1 Slider -->
-    <link name="l6l_finger_slider">
-        <inertial>
-            <mass value="0.001" />
-            <inertia ixx="0.000001" ixy="0" ixz="0" iyy="0.000001" iyz="0" izz="0.000001" />
-        </inertial>
-    </link>
-    <joint name="j7l1" type="prismatic">
-        <origin xyz="0.000 0.022 0.021" rpy="0 -1.572 0" />
-        <parent link="l6l_rail" />
-        <child link="l6l_finger_slider" />
-        <axis xyz="0 0 1" />
-        <limit lower="-0.02" upper="0.0" effort="1.0" velocity="0.1" />
-    </joint>
-    <!-- LEFT GRIPPER - Finger (actual mesh) -->
-    <link name="l6l_finger">
-        <inertial>
-            <origin xyz="0 0 0.015" rpy="0 0 0" />
-            <mass value="0.01" />
-            <inertia ixx="0.000001" ixy="0" ixz="0" iyy="0.000001" iyz="0" izz="0.000001" />
-        </inertial>
-        <visual>
-            <origin xyz="0 0 0" rpy="0 0 0" />
-            <geometry>
-                <mesh filename="package://dexter_arm_description/meshes/finger.stl" scale="0.001 0.001 0.001"/>
-            </geometry>
-            <material name="">
-                <color rgba="0.5 0.5 0.5 1" />
-            </material>
-        </visual>
-    </link>
-    <joint name="j6l_finger_fixed" type="fixed">
-        <origin xyz="0 0 0" rpy="0 0 0" />
-        <parent link="l6l_finger_slider" />
-        <child link="l6l_finger" />
-    </joint>
-    <!-- LEFT GRIPPER - Second Finger with Mimic Slider -->
-    <link name="l6l_finger2_slider">
-        <inertial>
-            <mass value="0.001" />
-            <inertia ixx="0.000001" ixy="0" ixz="0" iyy="0.000001" iyz="0" izz="0.000001" />
-        </inertial>
-    </link>
-    <joint name="j7l2" type="prismatic">
-        <origin xyz="0.060 0.022 0.021" rpy="0 1.572 0" />
-        <parent link="l6l_rail" />
-        <child link="l6l_finger2_slider" />
-        <axis xyz="0 0 1" />
-        <limit lower="-0.02" upper="0.0" effort="1.0" velocity="0.1" />
-    </joint>
-    <!-- LEFT GRIPPER - Second Finger (actual mesh) -->
-    <link name="l6l_finger2">
-        <inertial>
-            <origin xyz="0 0 0.015" rpy="0 0 0" />
-            <mass value="0.01" />
-            <inertia ixx="0.000001" ixy="0" ixz="0" iyy="0.000001" iyz="0" izz="0.000001" />
-        </inertial>
-        <visual>
-            <origin xyz="0 0 0" rpy="0 0 0" />
-            <geometry>
-                <mesh filename="package://dexter_arm_description/meshes/finger.stl" scale="0.001 0.001 0.001"/>
-            </geometry>
-            <material name="">
-                <color rgba="0.5 0.5 0.5 1" />
-            </material>
-        </visual>
-    </link>
-    <joint name="j6l_finger2_fixed" type="fixed">
-        <origin xyz="0 0 0" rpy="0 0 0" />
-        <parent link="l6l_finger2_slider" />
-        <child link="l6l_finger2" />
-    </joint>
-    <!-- LEFT ARM - Tool Center Point (TCP) -->
-    <link name="tool0_left">
-        <inertial>
-            <origin xyz="0 0 0" rpy="0 0 0" />
-            <mass value="0.001" />
-            <inertia ixx="0.000001" ixy="0" ixz="0" iyy="0.000001" iyz="0" izz="0.000001" />
-        </inertial>
-        <visual>
-            <origin xyz="0 0 0" rpy="0 0 0" />
-            <geometry>
-                <sphere radius="0.008" />
-            </geometry>
-            <material name="tcp_orange">
-                <color rgba="1.0 0.5 0.0 1.0" />
-            </material>
-        </visual>
-    </link>
-    <joint name="tool0_left_fixed_joint" type="fixed">
-        <origin xyz="0 0 -0.08" rpy="0 0 0" />
-        <parent link="l6l" />
-        <child link="tool0_left" />
-    </joint>
-    <!-- RIGHT ARM -->
-    <!-- Link l1r -->
-    <link name="l1r">
-        <inertial>
-            <origin xyz="2.06768076422351E-05 2.42861286636753E-17 -0.0236812970530664" rpy="0 0 0" />
-            <mass value="0.0412610106656879" />
-            <inertia ixx="6.45452263055137E-06" ixy="1.58739512138535E-22" ixz="5.67173895648283E-10"
-                     iyy="1.08529418395194E-05" iyz="2.01570916178023E-20" izz="8.35698735982533E-06" />
-        </inertial>
-        <visual>
-            <origin xyz="0 0 0" rpy="0 0 0" />
-            <geometry>
-                <mesh filename="package://dexter_arm_description/meshes/visual/l1r.STL" />
-            </geometry>
-            <material name="">
-                <color rgba="1 1 1 1" />
-            </material>
-        </visual>
-        <collision>
-            <origin xyz="0 0 0" rpy="0 0 0" />
-            <geometry>
-                <mesh filename="package://dexter_arm_description/meshes/collision/l1r.STL" />
-            </geometry>
-        </collision>
-    </link>
-    <joint name="j1r" type="revolute">
-        <origin xyz="0.185 0 0.4755" rpy="3.14159265358979 0 0" />
-        <parent link="base_link" />
-        <child link="l1r" />
-        <axis xyz="0 0 1" />
-        <limit lower="-1.57" upper="1.57" effort="343.0" velocity="5" />
-    </joint>
-    <!-- Link l2r -->
-    <link name="l2r">
-        <inertial>
-            <origin xyz="0.0419634783926228 0.00174598253548033 -0.000134261601576029" rpy="0 0 0" />
-            <mass value="0.0412639771770678" />
-            <inertia ixx="2.03907679743811E-05" ixy="-1.0944769820727E-07" ixz="8.41624870313865E-09"
-                     iyy="2.29316351108135E-05" iyz="-1.10603911559014E-06" izz="8.63338606000998E-06" />
-        </inertial>
-        <visual>
-            <origin xyz="0 0 0" rpy="0 0 0" />
-            <geometry>
-                <mesh filename="package://dexter_arm_description/meshes/visual/l2r.STL" />
-            </geometry>
-            <material name="">
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
File: src/dexter_arm_gazebo/urdf/dexter_arm_gazebo.xacro (robot description, xacro)
@@ -41,20 +41,28 @@
       <joint name="j7r1">
         <command_interface name="position"/>
-        <state_interface name="position"/>
+        <state_interface name="position">
+          <param name="initial_value">0.0</param>
+        </state_interface>
         <state_interface name="velocity"/>
       </joint>
       <joint name="j7r2">
         <command_interface name="position"/>
-        <state_interface name="position"/>
+        <state_interface name="position">
+          <param name="initial_value">-0.025</param>
+        </state_interface>
         <state_interface name="velocity"/>
       </joint>
       <joint name="j7l1">
         <command_interface name="position"/>
-        <state_interface name="position"/>
+        <state_interface name="position">
+          <param name="initial_value">-0.025</param>
+        </state_interface>
         <state_interface name="velocity"/>
       </joint>
       <joint name="j7l2">
         <command_interface name="position"/>
-        <state_interface name="position"/>
+        <state_interface name="position">
+          <param name="initial_value">0.0</param>
+        </state_interface>
         <state_interface name="velocity"/>
       </joint>
@@ -206,27 +214,15 @@
     </gazebo>
     <!-- Left Gripper Components -->
-    <gazebo reference="l6l_base1">
-        <material>Gazebo/Orange</material>
-    </gazebo>
-    <gazebo reference="l6l_rail">
-        <material>Gazebo/Orange</material>
-    </gazebo>
-    <gazebo reference="l6l_finger">
-        <material>Gazebo/Orange</material>
-    </gazebo>
-    <gazebo reference="l6l_finger2">
+    <gazebo reference="l7l1">
+        <material>Gazebo/Orange</material>
+    </gazebo>
+    <gazebo reference="l7l2">
         <material>Gazebo/Orange</material>
     </gazebo>
     <!-- Right Gripper Components -->
-    <gazebo reference="l6r_base1">
-        <material>Gazebo/Orange</material>
-    </gazebo>
-    <gazebo reference="l6r_rail">
-        <material>Gazebo/Orange</material>
-    </gazebo>
-    <gazebo reference="l6r_finger">
-        <material>Gazebo/Orange</material>
-    </gazebo>
-    <gazebo reference="l6r_finger2">
+    <gazebo reference="l7r1">
+        <material>Gazebo/Orange</material>
+    </gazebo>
+    <gazebo reference="l7r2">
         <material>Gazebo/Orange</material>
     </gazebo>
